Commit message: feat(gazebo): 双机仿真 RViz、Gazebo 传感器话题与文档更新
- sim_two_robots：robot_description 使用 ParameterValue(str)、xacro 传入 ros_namespace
- 安装并默认启动 two_robots_sim.rviz；可选 publish_world_tf 与 use_rviz
- mini_omni_robot.xacro：ROS2 ray/imu 插件 remapping 为 /scan 与 /imu
- README 补充话题、TF、下一步计划；增加 .gitignore 忽略 __pycache__

Made-with: Cursor

File: homo_multirobot_urdf/urdf/mini_omni_robot.xacro (robot description, xacro)
@@ -2,4 +2,7 @@
 <robot xmlns:xacro="http://www.ros.org/wiki/xacro" name="mini_omni_robot">
   <xacro:arg name="prefix" default=""/>
+  <xacro:arg name="use_gazebo" default="true"/>
+  <!-- 留空表示不额外设置；若 launch 里为每台机器人设置了命名空间，这里会把插件节点放进该 namespace -->
+  <xacro:arg name="ros_namespace" default=""/>
   <xacro:property name="p" value="$(arg prefix)"/>
   <link name="${p}base_footprint"/>
@@ -37,4 +40,16 @@
     </collision>
   </link>
+  <link name="${p}imu_link">
+    <inertial>
+      <origin xyz="0 0 0" rpy="0 0 0" />
+      <mass value="0.001" />
+      <inertia ixx="1e-6" ixy="0" ixz="0" iyy="1e-6" iyz="0" izz="1e-6" />
+    </inertial>
+  </link>
+  <joint name="${p}imu_joint" type="fixed">
+    <origin xyz="0 0 0" rpy="0 0 0" />
+    <parent link="${p}base_link" />
+    <child link="${p}imu_link" />
+  </joint>
   <link name="${p}front_wheel_link">
     <inertial>
@@ -241,3 +256,69 @@
     <axis xyz="0 0 0" />
   </joint>
+  <xacro:if value="$(arg use_gazebo)">
+    <!-- Ray lidar: publishes `<ns>/scan` -->
+    <gazebo reference="${p}laser_link">
+      <sensor name="${p}lidar" type="ray">
+        <always_on>true</always_on>
+        <update_rate>10</update_rate>
+        <visualize>true</visualize>
+        <ray>
+          <scan>
+            <horizontal>
+              <samples>720</samples>
+              <resolution>1</resolution>
+              <min_angle>-3.141592653589793</min_angle>
+              <max_angle>3.141592653589793</max_angle>
+            </horizontal>
+          </scan>
+          <range>
+            <min>0.12</min>
+            <max>12.0</max>
+            <resolution>0.01</resolution>
+          </range>
+          <noise>
+            <type>gaussian</type>
+            <mean>0.0</mean>
+            <stddev>0.01</stddev>
+          </noise>
+        </ray>
+        <!-- ROS2：默认话题为 ~/out；用 remapping 得到 /<ns>/scan，并用 LaserScan -->
+        <plugin name="${p}gazebo_ros_ray_sensor" filename="libgazebo_ros_ray_sensor.so">
+          <ros>
+            <namespace>$(arg ros_namespace)</namespace>
+            <remapping>~/out:=scan</remapping>
+          </ros>
+          <output_type>sensor_msgs/LaserScan</output_type>
+          <frame_name>${p}laser_link</frame_name>
+        </plugin>
+      </sensor>
+    </gazebo>
+    <!-- IMU: publishes `<ns>/imu` -->
+    <gazebo reference="${p}imu_link">
+      <sensor name="${p}imu" type="imu">
+        <always_on>true</always_on>
+        <update_rate>50</update_rate>
+        <visualize>false</visualize>
+        <imu>
+          <angular_velocity>
+            <x><noise type="gaussian"><mean>0.0</mean><stddev>0.0002</stddev></noise></x>
+            <y><noise type="gaussian"><mean>0.0</mean><stddev>0.0002</stddev></noise></y>
+            <z><noise type="gaussian"><mean>0.0</mean><stddev>0.0002</stddev></noise></z>
+          </angular_velocity>
+          <linear_acceleration>
+            <x><noise type="gaussian"><mean>0.0</mean><stddev>0.02</stddev></noise></x>
+            <y><noise type="gaussian"><mean>0.0</mean><stddev>0.02</stddev></noise></y>
+            <z><noise type="gaussian"><mean>0.0</mean><stddev>0.02</stddev></noise></z>
+          </linear_acceleration>
+        </imu>
+        <!-- ROS2：默认 ~/out；remapping 得到 /<ns>/imu -->
+        <plugin name="${p}gazebo_ros_imu_sensor" filename="libgazebo_ros_imu_sensor.so">
+          <ros>
+            <namespace>$(arg ros_namespace)</namespace>
+            <remapping>~/out:=imu</remapping>
+          </ros>
+        </plugin>
+      </sensor>
+    </gazebo>
+  </xacro:if>
 </robot>

Commit message: feat(sim): add ros2_control toggle for omni robot
Add use_ros2_control switch to mini_omni_robot xacro to select gazebo_ros2_control vs planar_move, and pass the flag through sim_two_robots.launch.py. Update READMEs with usage and verification steps.

File: homo_multirobot_urdf/urdf/mini_omni_robot.xacro (robot description, xacro)
@@ -3,7 +3,31 @@
   <xacro:arg name="prefix" default=""/>
   <xacro:arg name="use_gazebo" default="true"/>
+  <!-- true: use ros2_control + gazebo_ros2_control; false: fallback to gazebo_ros_planar_move -->
+  <xacro:arg name="use_ros2_control" default="false"/>
   <!-- 留空表示不额外设置；若 launch 里为每台机器人设置了命名空间，这里会把插件节点放进该 namespace -->
   <xacro:arg name="ros_namespace" default=""/>
   <xacro:property name="p" value="$(arg prefix)"/>
+  <xacro:if value="$(arg use_ros2_control)">
+    <ros2_control name="${p}mini_omni_robot_system" type="system">
+      <hardware>
+        <plugin>gazebo_ros2_control/GazeboSystem</plugin>
+      </hardware>
+      <joint name="${p}front_wheel_joint">
+        <command_interface name="velocity"/>
+        <state_interface name="position"/>
+        <state_interface name="velocity"/>
+      </joint>
+      <joint name="${p}left_wheel_joint">
+        <command_interface name="velocity"/>
+        <state_interface name="position"/>
+        <state_interface name="velocity"/>
+      </joint>
+      <joint name="${p}right_wheel_joint">
+        <command_interface name="velocity"/>
+        <state_interface name="position"/>
+        <state_interface name="velocity"/>
+      </joint>
+    </ros2_control>
+  </xacro:if>
   <link name="${p}base_footprint"/>
   <joint name="${p}base_footprint_joint" type="fixed">
@@ -322,17 +346,28 @@
     </gazebo>
     <!-- Planar move + odom: subscribes `<ns>/cmd_vel`, publishes `<ns>/odom` and TF -->
-    <gazebo>
-      <plugin name="${p}gazebo_ros_planar_move" filename="libgazebo_ros_planar_move.so">
-        <ros>
-          <namespace>$(arg ros_namespace)</namespace>
-        </ros>
-        <command_topic>cmd_vel</command_topic>
-        <odometry_topic>odom</odometry_topic>
-        <odometry_frame>${p}odom</odometry_frame>
-        <robot_base_frame>${p}base_footprint</robot_base_frame>
-        <publish_odom>true</publish_odom>
-        <publish_odom_tf>true</publish_odom_tf>
-      </plugin>
-    </gazebo>
+    <xacro:if value="$(arg use_ros2_control)">
+      <gazebo>
+        <plugin name="${p}gazebo_ros2_control" filename="libgazebo_ros2_control.so">
+          <ros>
+            <namespace>$(arg ros_namespace)</namespace>
+          </ros>
+        </plugin>
+      </gazebo>
+    </xacro:if>
+    <xacro:unless value="$(arg use_ros2_control)">
+      <gazebo>
+        <plugin name="${p}gazebo_ros_planar_move" filename="libgazebo_ros_planar_move.so">
+          <ros>
+            <namespace>$(arg ros_namespace)</namespace>
+          </ros>
+          <command_topic>cmd_vel</command_topic>
+          <odometry_topic>odom</odometry_topic>
+          <odometry_frame>${p}odom</odometry_frame>
+          <robot_base_frame>${p}base_footprint</robot_base_frame>
+          <publish_odom>true</publish_odom>
+          <publish_odom_tf>true</publish_odom_tf>
+        </plugin>
+      </gazebo>
+    </xacro:unless>
   </xacro:if>
 </robot>

Commit message: fix(sim): stop wheel sinking and yaw drift; inline empty world
- Simplify wheel collisions and tune wheel joint z to avoid initial ground penetration.
- Reduce wheel-ground friction in planar_move mode to prevent straight-line yaw drift.
- Inline sun/ground in empty.world to avoid model:// dependencies under restricted model paths/offline.
- Record findings and workarounds in urdf/gazebo README and BUG_RECORD.

Made-with: Cursor

File: homo_multirobot_urdf/urdf/mini_omni_robot.xacro (robot description, xacro)
@@ -8,4 +8,18 @@
   <xacro:arg name="ros_namespace" default=""/>
   <xacro:property name="p" value="$(arg prefix)"/>
+  <!-- Simple primitive collision (more stable than mesh collision in Gazebo) -->
+  <!-- base_link collision box size (meters) -->
+  <xacro:property name="base_collision_size_x" value="0.24"/>
+  <xacro:property name="base_collision_size_y" value="0.20"/>
+  <xacro:property name="base_collision_size_z" value="0.10"/>
+  <!-- wheel collision cylinder (meters): axis will be rotated to align with wheel joint axis -->
+  <!-- Keep consistent with controller config convention (often r=0.03) -->
+  <xacro:property name="wheel_collision_radius" value="0.03"/>
+  <xacro:property name="wheel_collision_width" value="0.020"/>
+  <!-- Small lift to avoid initial penetration / physics instability -->
+  <xacro:property name="wheel_collision_z_offset" value="0.007"/>
+  <!-- Gazebo contact: set wheel friction low to avoid yaw drift in planar_move mode -->
+  <xacro:property name="wheel_mu" value="0.0"/>
+  <xacro:property name="wheel_mu2" value="0.0"/>
   <xacro:if value="$(arg use_ros2_control)">
     <ros2_control name="${p}mini_omni_robot_system" type="system">
@@ -98,12 +112,14 @@
     </visual>
     <collision>
-      <origin xyz="0 0 0" rpy="0 0 0" />
-      <geometry>
-        <mesh filename="package://homo_multirobot_urdf/meshes/mini_omni_robot_meshes/front_wheel_link.STL" />
+      <!-- URDF cylinder axis is +Z; rotate to align with wheel joint axis (±Y) -->
+      <origin xyz="0 0 ${wheel_collision_z_offset}" rpy="1.57079632679 0 0" />
+      <geometry>
+        <cylinder radius="${wheel_collision_radius}" length="${wheel_collision_width}" />
       </geometry>
     </collision>
   </link>
   <joint name="${p}front_wheel_joint" type="continuous">
-    <origin xyz="0.10975 8.5571E-05 -0.0358" rpy="0 0 1.5708" />
+    <!-- z tuned to keep wheel above ground at spawn (avoid initial penetration) -->
+    <origin xyz="0.10975 8.5571E-05 -0.0300" rpy="0 0 1.5708" />
     <parent link="${p}base_link" />
     <child link="${p}front_wheel_link" />
@@ -132,12 +148,14 @@
     </visual>
     <collision>
-      <origin xyz="0 0 0" rpy="0 0 0" />
-      <geometry>
-        <mesh filename="package://homo_multirobot_urdf/meshes/mini_omni_robot_meshes/left_wheel_link.STL" />
+      <!-- URDF cylinder axis is +Z; rotate to align with wheel joint axis (±Y) -->
+      <origin xyz="0 0 ${wheel_collision_z_offset}" rpy="1.57079632679 0 0" />
+      <geometry>
+        <cylinder radius="${wheel_collision_radius}" length="${wheel_collision_width}" />
       </geometry>
     </collision>
   </link>
   <joint name="${p}left_wheel_joint" type="continuous">
-    <origin xyz="-0.054729 0.095045 -0.0358" rpy="0 0 -2.618" />
+    <!-- z tuned to keep wheel above ground at spawn (avoid initial penetration) -->
+    <origin xyz="-0.054729 0.095045 -0.0300" rpy="0 0 -2.618" />
     <parent link="${p}base_link" />
     <child link="${p}left_wheel_link" />
@@ -166,16 +184,31 @@
     </visual>
     <collision>
-      <origin xyz="0 0 0" rpy="0 0 0" />
-      <geometry>
-        <mesh filename="package://homo_multirobot_urdf/meshes/mini_omni_robot_meshes/right_wheel_link.STL" />
+      <!-- URDF cylinder axis is +Z; rotate to align with wheel joint axis (±Y) -->
+      <origin xyz="0 0 ${wheel_collision_z_offset}" rpy="1.57079632679 0 0" />
+      <geometry>
+        <cylinder radius="${wheel_collision_radius}" length="${wheel_collision_width}" />
       </geometry>
     </collision>
   </link>
   <joint name="${p}right_wheel_joint" type="continuous">
-    <origin xyz="-0.054729 -0.094874 -0.0358" rpy="0 0 -0.5236" />
+    <!-- z tuned to keep wheel above ground at spawn (avoid initial penetration) -->
+    <origin xyz="-0.054729 -0.094874 -0.0300" rpy="0 0 -0.5236" />
     <parent link="${p}base_link" />
     <child link="${p}right_wheel_link" />
     <axis xyz="0 -1 0" />
   </joint>
+  <!-- Gazebo wheel contact tuning (reduce unintended steering torque) -->
+  <gazebo reference="${p}front_wheel_link">
+    <mu1>${wheel_mu}</mu1>
+    <mu2>${wheel_mu2}</mu2>
+  </gazebo>
+  <gazebo reference="${p}left_wheel_link">
+    <mu1>${wheel_mu}</mu1>
+    <mu2>${wheel_mu2}</mu2>
+  </gazebo>
+  <gazebo reference="${p}right_wheel_link">
+    <mu1>${wheel_mu}</mu1>
+    <mu2>${wheel_mu2}</mu2>
+  </gazebo>
   <link name="${p}controller_link">
     <inertial>

Commit message: 新增双机 rf2o 里程计链路并完善仿真参数与文档
- 引入 rf2o_laser_odometry（ROS2）并提供双机启动与 TF 开关
- sim_two_robots 支持 world_name 从本包 worlds 选择世界文件
- 修复 laser_link 180° 翻转导致 rf2o 速度符号反号
- 更新各包 README/BUG_RECORD，清理不再使用的 rf2o 参数 yaml

File: homo_multirobot_urdf/urdf/mini_omni_robot.xacro (robot description, xacro)
@@ -7,4 +7,7 @@
   <!-- 留空表示不额外设置；若 launch 里为每台机器人设置了命名空间，这里会把插件节点放进该 namespace -->
   <xacro:arg name="ros_namespace" default=""/>
+  <!-- gazebo_ros_planar_move: toggle odom topic / TF publication -->
+  <xacro:arg name="planar_publish_odom" default="true"/>
+  <xacro:arg name="planar_publish_odom_tf" default="true"/>
   <xacro:property name="p" value="$(arg prefix)"/>
   <!-- Simple primitive collision (more stable than mesh collision in Gazebo) -->
@@ -274,5 +277,5 @@
   </link>
   <joint name="${p}laser_joint" type="fixed">
-    <origin xyz="0.005095 8.5571E-05 0.097524" rpy="0 0 3.1416" />
+    <origin xyz="0.005095 8.5571E-05 0.097524" rpy="0 0 0" />
     <parent link="${p}base_link" />
     <child link="${p}laser_link" />
@@ -398,6 +401,6 @@
           <odometry_frame>${p}odom</odometry_frame>
           <robot_base_frame>${p}base_footprint</robot_base_frame>
-          <publish_odom>true</publish_odom>
-          <publish_odom_tf>true</publish_odom_tf>
+          <publish_odom>$(arg planar_publish_odom)</publish_odom>
+          <publish_odom_tf>$(arg planar_publish_odom_tf)</publish_odom_tf>
         </plugin>
       </gazebo>

Commit message: 新增实机单机 rf2o 启动并统一仿真/可视化外观
- homo_multirobot_localization 新增 rf2o_single_robot.launch.py，支持 namespace/prefix 等参数用于实机部署
- 更新仓库级与包级 README，补充实机单机 rf2o 启动与参数说明
- 优化 mini_omni_robot 在 Gazebo/RViz 的材质与配色（底盘深灰、控制板 PCB 绿、传感器深色）

File: homo_multirobot_urdf/urdf/mini_omni_robot.xacro (robot description, xacro)
@@ -71,5 +71,5 @@
       </geometry>
       <material name="">
-        <color rgba="0.741176470588235 0.901960784313726 0.956862745098039 1" />
+        <color rgba="0.22 0.22 0.22 1" />
       </material>
     </visual>
@@ -111,5 +111,5 @@
       </geometry>
       <material name="">
-        <color rgba="0.376470588235294 0.376470588235294 0.376470588235294 1" />
+        <color rgba="0.18 0.18 0.18 1" />
       </material>
     </visual>
@@ -147,5 +147,5 @@
       </geometry>
       <material name="">
-        <color rgba="0.376470588235294 0.376470588235294 0.376470588235294 1" />
+        <color rgba="0.18 0.18 0.18 1" />
       </material>
     </visual>
@@ -183,5 +183,5 @@
       </geometry>
       <material name="">
-        <color rgba="0.376470588235294 0.376470588235294 0.376470588235294 1" />
+        <color rgba="0.18 0.18 0.18 1" />
       </material>
     </visual>
@@ -205,12 +205,43 @@
     <mu1>${wheel_mu}</mu1>
     <mu2>${wheel_mu2}</mu2>
+    <material>Gazebo/DarkGrey</material>
+    <ambient>0.08 0.08 0.08 1</ambient>
+    <diffuse>0.18 0.18 0.18 1</diffuse>
+    <specular>0.15 0.15 0.15 1</specular>
   </gazebo>
   <gazebo reference="${p}left_wheel_link">
     <mu1>${wheel_mu}</mu1>
     <mu2>${wheel_mu2}</mu2>
+    <material>Gazebo/DarkGrey</material>
+    <ambient>0.08 0.08 0.08 1</ambient>
+    <diffuse>0.18 0.18 0.18 1</diffuse>
+    <specular>0.15 0.15 0.15 1</specular>
   </gazebo>
   <gazebo reference="${p}right_wheel_link">
     <mu1>${wheel_mu}</mu1>
     <mu2>${wheel_mu2}</mu2>
+    <material>Gazebo/DarkGrey</material>
+    <ambient>0.08 0.08 0.08 1</ambient>
+    <diffuse>0.18 0.18 0.18 1</diffuse>
+    <specular>0.15 0.15 0.15 1</specular>
+  </gazebo>
+  <!-- Gazebo materials (visual polish) -->
+  <gazebo reference="${p}base_link">
+    <material>Gazebo/Grey</material>
+    <ambient>0.10 0.10 0.10 1</ambient>
+    <diffuse>0.22 0.22 0.22 1</diffuse>
+    <specular>0.35 0.35 0.35 1</specular>
+  </gazebo>
+  <gazebo reference="${p}controller_link">
+    <material>Gazebo/Green</material>
+    <ambient>0.02 0.08 0.04 1</ambient>
+    <diffuse>0.06 0.35 0.18 1</diffuse>
+    <specular>0.20 0.25 0.20 1</specular>
+  </gazebo>
+  <gazebo reference="${p}camera_link">
+    <material>Gazebo/Black</material>
+    <ambient>0.02 0.02 0.02 1</ambient>
+    <diffuse>0.08 0.08 0.08 1</diffuse>
+    <specular>0.25 0.25 0.25 1</specular>
   </gazebo>
   <link name="${p}controller_link">
@@ -232,5 +263,5 @@
       </geometry>
       <material name="">
-        <color rgba="0.741176470588235 0.901960784313726 0.956862745098039 1" />
+        <color rgba="0.06 0.35 0.18 1" />
       </material>
     </visual>
@@ -266,5 +297,5 @@
       </geometry>
       <material name="">
-        <color rgba="0.376470588235294 0.376470588235294 0.376470588235294 1" />
+        <color rgba="0.08 0.08 0.08 1" />
       </material>
     </visual>
@@ -300,5 +331,5 @@
       </geometry>
       <material name="">
-        <color rgba="1 1 1 1" />
+        <color rgba="0.08 0.08 0.08 1" />
       </material>
     </visual>
@@ -319,4 +350,8 @@
     <!-- Ray lidar: publishes `<ns>/scan` -->
     <gazebo reference="${p}laser_link">
+      <material>Gazebo/Black</material>
+      <ambient>0.05 0.05 0.05 1</ambient>
+      <diffuse>0.12 0.12 0.12 1</diffuse>
+      <specular>0.20 0.20 0.20 1</specular>
       <sensor name="${p}lidar" type="ray">
         <always_on>true</always_on>
