Commit message: feat: 新增齐次控制编队算法 C++ 实现 + slam_toolbox 纯定位支持
新增:
- homo_multirobot_formation_control: 齐次控制 Leader-Follower 编队算法 (C++/Eigen)
  包括 hnorm (二分法)、lpc2hpc (LPC→HPC 升级)、双重积分器控制器
  通过 TF + EKF odometry/filtered 获取状态，兼容 AMCL/slam_toolbox 定位
  支持单/双 follower launch 文件，带参数化配置
- homo_multirobot_nav: 新增 slam_toolbox 纯定位 launch (slam_toolbox_loc_*)
  比 AMCL 粒子滤波更平滑，适合编队控制联调
- leader_control.py: 领航者正弦轨迹生成节点

修改:
- mini_omni_robot.xacro: 底盘总质量 0.58kg→2.0kg (匹配论文，质量+惯量等比例缩放)
- 项目 README: 新增 formation_control、slam_toolbox 定位章节
- homo_multirobot_nav README: 补充 slam_toolbox 定位启动方式

关键 bug 修复 (详见 BUG_RECORD.md):
- Eigen 3.4 API 适配 (expm→.exp(), sqrtm→.sqrt(), aliasing 规避)
- trans_con 固定尺寸矩阵死循环 (改用 MatrixXd)
- c clamp 0.1→0.5 抑制定位噪声非线性放大
- val_a/val_b 比值 clamp 防止增益爆炸

File: homo_multirobot_urdf/urdf/mini_omni_robot.xacro (robot description, xacro)
@@ -56,12 +56,12 @@
     <inertial>
       <origin xyz="-0.00215152015512567 -0.00354771497616371 -0.00238850986636495" rpy="0 0 0" />
-      <mass value="0.316971084822964" />
-      <inertia
-        ixx="0.000420307413554536"
-        ixy="8.53304678996615E-07"
-        ixz="3.25484281157172E-11"
-        iyy="0.000423240319736897"
+      <mass value="1.097575775416477e+00" />
+      <inertia
+        ixx="1.455398480915292e-03"
+        ixy="2.954738111961579e-06"
+        ixz="1.127054420362940e-10"
+        iyy="1.465554255152953e-03"
         iyz="-2.92206846665081E-11"
-        izz="0.000803923344739989" />
+        izz="2.783745365831159e-03" />
     </inertial>
     <visual>
@@ -84,6 +84,6 @@
     <inertial>
       <origin xyz="0 0 0" rpy="0 0 0" />
-      <mass value="0.001" />
-      <inertia ixx="1e-6" ixy="0" ixz="0" iyy="1e-6" iyz="0" izz="1e-6" />
+      <mass value="3.462700000000000e-03" />
+      <inertia ixx="3.462700000000000e-06" ixy="0.000000000000000e+00" ixz="0.000000000000000e+00" iyy="3.462700000000000e-06" iyz="0.000000000000000e+00" izz="3.462700000000000e-06" />
     </inertial>
   </link>
@@ -96,12 +96,12 @@
     <inertial>
       <origin xyz="5.74714974423331E-05 0.00320699063859495 -4.61768854820438E-05" rpy="0 0 0" />
-      <mass value="0.0418742906509581" />
-      <inertia
-        ixx="1.11530020202845E-05"
-        ixy="2.36675244306518E-08"
+      <mass value="1.449981062370726e-01" />
+      <inertia
+        ixx="3.861950009563913e-05"
+        ixy="8.195353684601798e-08"
         ixz="-5.43279459256917E-08"
-        iyy="1.8768089937325E-05"
+        iyy="6.498826502597528e-05"
         iyz="-4.01883681793204E-08"
-        izz="1.11464768270902E-05" />
+        izz="3.859690530916523e-05" />
     </inertial>
     <visual>
@@ -132,12 +132,12 @@
     <inertial>
       <origin xyz="5.74678573044898E-05 0.00320699471167032 -4.61750060654284E-05" rpy="0 0 0" />
-      <mass value="0.041874288756166" />
-      <inertia
-        ixx="1.11530017211417E-05"
-        ixy="2.36641581685783E-08"
+      <mass value="1.449980996759760e-01" />
+      <inertia
+        ixx="3.861949905979736e-05"
+        ixy="8.194188049033608e-08"
         ixz="-5.43274481797102E-08"
-        iyy="1.87681100612576E-05"
+        iyy="6.498833470911669e-05"
         iyz="-4.01888165769215E-08"
-        izz="1.11464785833887E-05" />
+        izz="3.859691139070005e-05" />
     </inertial>
     <visual>
@@ -168,12 +168,12 @@
     <inertial>
       <origin xyz="5.74721854603097E-05 0.00320699380279695 -4.61761038215297E-05" rpy="0 0 0" />
-      <mass value="0.0418742868228469" />
-      <inertia
-        ixx="1.11530020877519E-05"
-        ixy="2.36755527469659E-08"
+      <mass value="1.449980929814720e-01" />
+      <inertia
+        ixx="3.861950032925850e-05"
+        ixy="8.198133649691883e-08"
         ixz="-5.43278673691997E-08"
-        iyy="1.87681107970762E-05"
+        iyy="6.498833725703576e-05"
         iyz="-4.0189135655947E-08"
-        izz="1.11464784876816E-05" />
+        izz="3.859691105929508e-05" />
     </inertial>
     <visual>
@@ -248,12 +248,12 @@
     <inertial>
       <origin xyz="-0.0166307508329173 0.0377059276016881 0.0221732694812525" rpy="0 0 0" />
-      <mass value="0.0388361502106471" />
-      <inertia
-        ixx="2.23207514180048E-05"
-        ixy="9.5272750875175E-07"
+      <mass value="1.344779373344077e-01" />
+      <inertia
+        ixx="7.729006593512523e-05"
+        ixy="3.299009544554685e-06"
         ixz="-5.84384794338806E-08"
-        iyy="2.46082780117255E-05"
-        iyz="3.14216783338302E-07"
-        izz="4.60494109024797E-05" />
+        iyy="8.521108427120188e-05"
+        iyz="1.088038455665538e-06"
+        izz="1.594552951320165e-04" />
     </inertial>
     <visual>
@@ -282,12 +282,12 @@
     <inertial>
       <origin xyz="0.0023946067243534 -4.3623586159597E-06 0.00454035676315102" rpy="0 0 0" />
-      <mass value="0.0391766918292892" />
-      <inertia
-        ixx="2.82296075691487E-05"
+      <mass value="1.356571307972797e-01" />
+      <inertia
+        ixx="9.775066212969120e-05"
         ixy="-2.19900290000419E-09"
-        ixz="1.07118438746105E-06"
-        iyy="3.37984497834087E-05"
-        iyz="6.83963658170686E-10"
-        izz="4.50920076493152E-05" />
+        ixz="3.709190178461378e-06"
+        iyy="1.170338920650093e-04"
+        iyz="2.368360959147634e-09"
+        izz="1.561400948872837e-04" />
     </inertial>
     <visual>
@@ -316,12 +316,12 @@
     <inertial>
       <origin xyz="-1.30544696302914E-07 -9.32154475080064E-08 1.07624265707762E-07" rpy="0 0 0" />
-      <mass value="0.0559842512081409" />
-      <inertia
-        ixx="0.000130810959339877"
-        ixy="1.20255128069094E-07"
-        ixz="1.62335437079563E-06"
-        iyy="1.91148634968207E-05"
+      <mass value="1.938566666584295e-01" />
+      <inertia
+        ixx="4.529591089061920e-04"
+        ixy="4.164074319648517e-07"
+        ixz="5.621189179754027e-06"
+        iyy="6.618903783044104e-05"
         iyz="-2.80016756154036E-08"
-        izz="0.00013138746952371" />
+        izz="4.549553907197507e-04" />
     </inertial>
     <visual>
@@ -356,5 +356,5 @@
       <sensor name="${p}lidar" type="ray">
         <always_on>true</always_on>
-        <update_rate>10</update_rate>
+        <update_rate>15</update_rate>
         <visualize>true</visualize>
         <ray>

Commit message: 部署 turn_on_wheeltec_robot 适配 mini_omni 多机运行
- 添加实车驱动依赖包: serial_ros2, wheeltec_robot_msg, lslidar_ros2
- 精简 turn_on_wheeltec_robot: 仅支持 mini_omni / N10 雷达 / STM32 IMU
- 新建 bringup_mini_omni.launch.py 支持 namespace/prefix 多机隔离
- 删除冗余: 36个其他车型配置、相机/EKF launch、未使用的 msg
- xacro 添加 gyro_link / laser 别名 link 兼容 Wheeltec 驱动帧名
- ImuProcessor 话题路径改为相对路径适配 namespace

File: homo_multirobot_urdf/urdf/mini_omni_robot.xacro (robot description, xacro)
@@ -93,4 +93,11 @@
     <child link="${p}imu_link" />
   </joint>
+  <!-- 别名：gyro_link（Wheeltec 驱动使用），挂在 imu_link 下，0 偏移 -->
+  <link name="${p}gyro_link"/>
+  <joint name="${p}gyro_alias_joint" type="fixed">
+    <origin xyz="0 0 0" rpy="0 0 0"/>
+    <parent link="${p}imu_link"/>
+    <child link="${p}gyro_link"/>
+  </joint>
   <link name="${p}front_wheel_link">
     <inertial>
@@ -312,4 +319,11 @@
     <child link="${p}laser_link" />
     <axis xyz="0 0 0" />
+  </joint>
+  <!-- 别名：laser（Wheeltec 驱动使用），挂在 laser_link 下，0 偏移 -->
+  <link name="${p}laser"/>
+  <joint name="${p}laser_alias_joint" type="fixed">
+    <origin xyz="0 0 0" rpy="0 0 0"/>
+    <parent link="${p}laser_link"/>
+    <child link="${p}laser"/>
   </joint>
   <link name="${p}camera_link">
